Commit message: Configuration and addition of gmapping and configuration of the posiition LiDAR on the robot.

File: robots/pioneer3at_body.xacro (robot description, xacro)
@@ -157,5 +157,5 @@
     </collision>
     <visual>
-      <origin xyz="0.105 0 0.07" rpy="0 0 0"/>
+      <origin xyz="0.030 0 0.0" rpy="0 0 0"/>
       <geometry>
         <mesh filename="package://mapping_pioneer3at/meshes/hokuyo1.dae"/>
@@ -186,7 +186,6 @@
         <range>
           <min>0.10</min>
-          <!--<max>10.0</max> ORIGINAL ESTO PARA DEJAR MENOS ESPACIOS AL SENSAR-->
-          <max>80.0</max>
-          <resolution>0.01</resolution>  <!-- 10 mm/± 15 mm -->
+          <max>30.0</max>
+          <resolution>0.01</resolution>
         </range>
         <noise>

Commit message: adding trajectory and class navigation

File: robots/pioneer3at_body.xacro (robot description, xacro)
@@ -151,5 +151,5 @@
   <link name="hokuyo_link">
     <collision>
-      <origin xyz="0.105 0 0.10" rpy="0 0 0"/>
+      <origin xyz="0.030 0 0.0" rpy="0 0 0"/>
       <geometry>
     <box size="0.01 0.01 0.01"/>
